File: RP2354 Schematic.kicad_sch (KiCad schematic)
At the start: 27 parts, among them J1 Conn_01x03, SW1 SW_Push, U1 RP2350A-QFN60, Y1 ABM8-272-T3

Commit message: Test Change
Other:
- note added: "THIS IS A TEST OF GITHUB THROUGH KICAD"
Changed lines of the file:
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@@
 	(generator_version "9.0")
 	(paper "A4")
+	(text "THIS IS A TEST OF GITHUB THROUGH KICAD"
+		(exclude_from_sim no)
+		(at 202.946 128.27 0)
+		(effects
+			(font
+				(size 1.27 1.27)
+			)
+		)
+	)
 	(text "USB connection"
 		(exclude_from_sim no)
